File: Hardware/esp-oled-thing.brd (EAGLE design)
At the start: 48.3 x 27 mm, 44 parts, among them Q1 2.5A/30V, U1 MCP73831, U2 TPS61200

Commit message: more layout progress
Routing:
- net N$4: track 0.00 -> 52.6 mm, vias 0 -> 1
- net N$8: track 0.00 -> 50.7 mm, vias 0 -> 1
- net VBATT: track 7.74 -> 50.1 mm, vias 0 -> 1
- net N$2: track 0.00 -> 22.0 mm
- net CHARGER_STATUS: track 0.00 -> 9.70 mm
- net N$20: track 0.00 -> 7.72 mm
- net SDA: track 0.00 -> 7.60 mm
- net SCL: track 0.00 -> 7.31 mm
- net N$19: track 0.00 -> 7.26 mm
- net N$1: track 0.00 -> 6.23 mm
- net 5VIN: track 21.6 -> 26.1 mm
- net POWERPATH_OUT: track 0.00 -> 2.25 mm
Changed lines of the file:
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@@
 <vertex x="0" y="26.924"/>
 </polygon>
+<wire x1="33.528" y1="16.51" x2="32.79" y2="16.76" width="0" layer="19" extent="1-1"/>
 <wire x1="35.79" y1="16.76" x2="35.052" y2="16.51" width="0" layer="19" extent="1-1"/>
-<wire x1="32.79" y1="16.76" x2="33.528" y2="16.51" width="0" layer="19" extent="1-1"/>
+<wire x1="27.432" y1="17.159" x2="30.988" y2="15.89" width="0" layer="19" extent="1-1"/>
 </signal>
 <signal name="SCL">
@@
 <contactref element="BOOTL" pad="4"/>
 <contactref element="I2C_OLED" pad="3"/>
+<wire x1="10.09" y1="20.87" x2="10.09" y2="15.94" width="0.4064" layer="16"/>
+<wire x1="10.09" y1="15.94" x2="11.77" y2="14.26" width="0.4064" layer="16"/>
 <wire x1="10.09" y1="20.87" x2="16.204" y2="24.738" width="0" layer="19" extent="1-1"/>
-<wire x1="11.77" y1="14.26" x2="10.09" y2="20.87" width="0" layer="19" extent="16-16"/>
 <wire x1="17.63" y1="4.725" x2="11.77" y2="14.26" width="0" layer="19" extent="16-16"/>
 <wire x1="22.71" y1="4.725" x2="17.63" y2="4.725" width="0" layer="19" extent="16-16"/>
@@
 <contactref element="I2C_OLED" pad="4"/>
 <contactref element="GPIO2_GND" pad="2"/>
+<wire x1="12.09" y1="20.87" x2="12.09" y2="16.92" width="0.4064" layer="16"/>
+<wire x1="12.09" y1="16.92" x2="14.67" y2="14.34" width="0.4064" layer="16"/>
 <wire x1="18.744" y1="24.738" x2="22.294" y2="24.638" width="0" layer="19" extent="1-1"/>
 <wire x1="12.09" y1="20.87" x2="18.744" y2="24.738" width="0" layer="19" extent="1-1"/>
-<wire x1="14.67" y1="14.34" x2="12.09" y2="20.87" width="0" layer="19" extent="16-16"/>
 </signal>
 <signal name="VCC">
@@
 <contactref element="U$2" pad="TX"/>
 <contactref element="R3" pad="1"/>
-<wire x1="3.95" y1="14.38" x2="2.09" y2="20.87" width="0" layer="19" extent="16-16"/>
+<wire x1="2.09" y1="20.87" x2="2.09" y2="16.24" width="0.4064" layer="16"/>
+<wire x1="2.09" y1="16.24" x2="3.95" y2="14.38" width="0.4064" layer="16"/>
 </signal>
 <signal name="N$20">
 <contactref element="U$2" pad="RX"/>
 <contactref element="R4" pad="1"/>
-<wire x1="6.87" y1="14.3" x2="4.09" y2="20.87" width="0" layer="19" extent="16-16"/>
+<wire x1="4.09" y1="20.87" x2="4.09" y2="17.08" width="0.4064" layer="16"/>
+<wire x1="4.09" y1="17.08" x2="6.87" y2="14.3" width="0.4064" layer="16"/>
 </signal>
 <signal name="RST">
@@
 <contactref element="UART" pad="2"/>
 <contactref element="R3" pad="2"/>
-<wire x1="3.95" y1="12.48" x2="41.894" y2="2.286" width="0" layer="19" extent="16-16"/>
+<wire x1="3.95" y1="12.48" x2="3.95" y2="8.776" width="0.4064" layer="16"/>
+<wire x1="3.95" y1="8.776" x2="3.048" y2="7.874" width="0.4064" layer="16"/>
+<wire x1="3.048" y1="7.874" x2="3.048" y2="2.54" width="0.4064" layer="16"/>
+<via x="3.048" y="2.54" extent="1-16" drill="0.6"/>
+<wire x1="3.048" y1="2.54" x2="36.068" y2="2.54" width="0.4064" layer="1"/>
+<wire x1="36.068" y1="2.54" x2="38.608" y2="5.08" width="0.4064" layer="1"/>
+<wire x1="38.608" y1="5.08" x2="41.148" y2="5.08" width="0.4064" layer="1"/>
+<wire x1="41.148" y1="5.08" x2="41.656" y2="4.572" width="0.4064" layer="1"/>
+<wire x1="41.656" y1="4.572" x2="41.656" y2="2.524" width="0.4064" layer="1"/>
+<wire x1="41.656" y1="2.524" x2="41.894" y2="2.286" width="0.4064" layer="1"/>
 </signal>
 <signal name="N$8">
 <contactref element="UART" pad="3"/>
 <contactref element="R4" pad="2"/>
-<wire x1="6.87" y1="12.4" x2="44.434" y2="2.286" width="0" layer="19" extent="16-16"/>
+<wire x1="6.87" y1="12.4" x2="7.574" y2="12.4" width="0.4064" layer="16"/>
+<wire x1="7.574" y1="12.4" x2="7.62" y2="12.446" width="0.4064" layer="16"/>
+<wire x1="7.62" y1="12.446" x2="7.62" y2="8.382" width="0.4064" layer="16"/>
+<wire x1="7.62" y1="8.382" x2="7.112" y2="7.874" width="0.4064" layer="16"/>
+<wire x1="7.112" y1="7.874" x2="7.112" y2="4.064" width="0.4064" layer="16"/>
+<wire x1="7.112" y1="4.064" x2="7.366" y2="3.81" width="0.4064" layer="16"/>
+<via x="7.366" y="3.81" extent="1-16" drill="0.6"/>
+<wire x1="7.366" y1="3.81" x2="36.068" y2="3.81" width="0.4064" layer="1"/>
+<wire x1="36.068" y1="3.81" x2="38.608" y2="6.35" width="0.4064" layer="1"/>
+<wire x1="38.608" y1="6.35" x2="42.418" y2="6.35" width="0.4064" layer="1"/>
+<wire x1="42.418" y1="6.35" x2="44.45" y2="4.318" width="0.4064" layer="1"/>
+<wire x1="44.45" y1="4.318" x2="44.45" y2="2.302" width="0.4064" layer="1"/>
+<wire x1="44.45" y1="2.302" x2="44.434" y2="2.286" width="0.4064" layer="1"/>
 </signal>
 <signal name="N$13">
@@
 <wire x1="26.416" y1="5.588" x2="26.416" y2="6.5079" width="0.3048" layer="1"/>
 <wire x1="26.416" y1="6.5079" x2="26.482" y2="6.5739" width="0.3048" layer="1"/>
-<wire x1="41.926" y1="23.048" x2="42.606" y2="25.146" width="0" layer="19" extent="1-1"/>
-<wire x1="39.878" y1="23.248" x2="41.926" y2="23.048" width="0" layer="19" extent="1-1"/>
+<wire x1="41.926" y1="23.048" x2="42.606" y2="23.728" width="0.3048" layer="1"/>
+<wire x1="42.606" y1="23.728" x2="42.606" y2="25.146" width="0.3048" layer="1"/>
+<wire x1="41.926" y1="23.048" x2="41.726" y2="23.248" width="0.3048" layer="1"/>
+<wire x1="41.726" y1="23.248" x2="39.878" y2="23.248" width="0.3048" layer="1"/>
 <wire x1="41.722" y1="12.162" x2="41.926" y2="23.048" width="0" layer="19" extent="1-1"/>
 <wire x1="24.384" y1="7.253" x2="26.416" y2="6.5079" width="0" layer="19" extent="1-1"/>
@@
 <wire x1="22.794" y1="16.256" x2="22.86" y2="16.256" width="0.3048" layer="1"/>
 <wire x1="22.86" y1="16.256" x2="22.86" y2="16.002" width="0.3048" layer="1"/>
-<wire x1="44.026" y1="22.098" x2="47.03" y2="25.044" width="0" layer="19" extent="1-1"/>
-<wire x1="32.766" y1="8.128" x2="44.026" y2="22.098" width="0" layer="19" extent="1-1"/>
-<wire x1="23.763" y1="11.43" x2="26.416" y2="9.1081" width="0" layer="19" extent="1-1"/>
-<wire x1="22.86" y1="16.002" x2="23.763" y2="11.43" width="0" layer="19" extent="1-1"/>
+<wire x1="47.03" y1="25.044" x2="46.972" y2="25.044" width="0.4064" layer="1"/>
+<wire x1="46.972" y1="25.044" x2="44.026" y2="22.098" width="0.8128" layer="1"/>
+<wire x1="32.766" y1="8.128" x2="32.766" y2="6.604" width="0.8128" layer="1"/>
+<via x="32.766" y="6.604" extent="1-16" drill="0.6" shape="square"/>
+<wire x1="32.766" y1="6.604" x2="33.02" y2="6.858" width="0.8128" layer="16"/>
+<wire x1="33.02" y1="6.858" x2="33.02" y2="12.192" width="0.8128" layer="16"/>
+<wire x1="33.02" y1="12.192" x2="34.29" y2="13.462" width="0.8128" layer="16"/>
+<wire x1="34.29" y1="13.462" x2="36.576" y2="13.462" width="0.8128" layer="16"/>
+<wire x1="36.576" y1="13.462" x2="39.116" y2="16.002" width="0.8128" layer="16"/>
+<wire x1="39.116" y1="16.002" x2="39.116" y2="20.574" width="0.8128" layer="16"/>
+<wire x1="39.116" y1="20.574" x2="40.64" y2="22.098" width="0.8128" layer="16"/>
+<wire x1="40.64" y1="22.098" x2="44.026" y2="22.098" width="0.8128" layer="16"/>
+<wire x1="44.026" y1="22.098" x2="46.972" y2="25.044" width="0.8128" layer="16"/>
+<wire x1="46.972" y1="25.044" x2="47.03" y2="25.044" width="0.8128" layer="16"/>
+<wire x1="22.86" y1="16.002" x2="24.13" y2="14.732" width="0.4064" layer="1"/>
+<wire x1="24.13" y1="14.732" x2="24.13" y2="12.446" width="0.4064" layer="1"/>
+<wire x1="24.13" y1="12.446" x2="23.763" y2="12.079" width="0.4064" layer="1"/>
+<wire x1="23.763" y1="12.079" x2="23.763" y2="11.43" width="0.4064" layer="1"/>
+<wire x1="23.763" y1="11.43" x2="26.0189" y2="9.1741" width="0.4064" layer="1"/>
+<wire x1="26.0189" y1="9.1741" x2="26.482" y2="9.1741" width="0.4064" layer="1"/>
 </signal>
 <signal name="N$14">
@@
 <contactref element="U1" pad="1"/>
 <contactref element="CHARGER_STATUS" pad="1"/>
-<wire x1="20.008" y1="6.604" x2="28.382" y2="9.1741" width="0" layer="19" extent="1-1"/>
+<wire x1="20.008" y1="6.604" x2="21.59" y2="6.604" width="0.4064" layer="1"/>
+<wire x1="21.59" y1="6.604" x2="24.638" y2="3.556" width="0.4064" layer="1"/>
+<wire x1="24.638" y1="3.556" x2="28.448" y2="3.556" width="0.4064" layer="1"/>
+<wire x1="28.448" y1="3.556" x2="28.382" y2="9.1741" width="0" layer="19" extent="1-1"/>
 </signal>
 <signal name="VIN">
@@
 <contactref element="Q1" pad="2"/>
 <contactref element="SJ5" pad="3"/>
-<wire x1="39.878" y1="20.948" x2="41.926" y2="21.148" width="0" layer="19" extent="1-1"/>
+<wire x1="39.878" y1="20.948" x2="41.926" y2="20.948" width="0.4064" layer="1"/>
+<wire x1="41.926" y1="20.948" x2="41.926" y2="21.148" width="0.4064" layer="1"/>
 <wire x1="35.814" y1="8.128" x2="39.878" y2="20.948" width="0" layer="19" extent="1-1"/>
 </signal>
@@
 <contactref element="CHARGER_STATUS" pad="2"/>
 <contactref element="U$2" pad="GPIO13"/>
-<wire x1="14.09" y1="6.87" x2="19.108" y2="6.604" width="0" layer="19" extent="1-1"/>
+<wire x1="14.09" y1="6.87" x2="14.09" y2="6.978" width="0.4064" layer="1"/>
+<wire x1="14.09" y1="6.978" x2="15.24" y2="8.128" width="0.4064" layer="1"/>
+<wire x1="15.24" y1="8.128" x2="17.584" y2="8.128" width="0.4064" layer="1"/>
+<wire x1="17.584" y1="8.128" x2="19.108" y2="6.604" width="0.4064" layer="1"/>
 </signal>
 <signal name="N$2">
@@
 <contactref element="R14" pad="1"/>
 <contactref element="R15" pad="2"/>
-<wire x1="20.894" y1="13.97" x2="20.894" y2="16.256" width="0" layer="19" extent="1-1"/>
-<wire x1="4.09" y1="6.87" x2="20.894" y2="13.97" width="0" layer="19" extent="1-1"/>
+<wire x1="20.894" y1="13.97" x2="20.894" y2="16.256" width="0.4064" layer="1"/>
+<wire x1="20.894" y1="13.97" x2="16.322" y2="9.398" width="0.4064" layer="1"/>
+<wire x1="16.322" y1="9.398" x2="6.618" y2="9.398" width="0.4064" layer="1"/>
+<wire x1="6.618" y1="9.398" x2="4.09" y2="6.87" width="0.4064" layer="1"/>
 </signal>
 <signal name="N$3">

Commit message: more layout progress, some optimisation needed in the layout.
Parts:
- moved R6 11.0 mm to (30.2, 5.84), turned to 0 degrees
- moved S1 0.25 mm to (5.08, 24.6)
- turned GPIO2_GND to 180 degrees
Routing:
- net VCC: track 29.9 -> 76.1 mm, vias 0 -> 1
- net SCL: track 7.31 -> 46.1 mm
- net TPS_EN: track 2.06 -> 31.2 mm, vias 0 -> 1
- net N$3: track 0.00 -> 27.3 mm, vias 0 -> 1
- net N$5: track 0.00 -> 21.4 mm
- net 5VIN: track 26.1 -> 46.9 mm, vias 0 -> 4
- net N$13: track 16.9 -> 1.50 mm
- net POWERPATH_OUT: track 2.25 -> 16.8 mm
- net RST: track 0.00 -> 13.8 mm
- net VBATT: track 50.1 -> 54.0 mm
- net CHARGER_STATUS: track 9.70 -> 13.6 mm, vias 0 -> 2
- net GND: track 33.6 -> 30.5 mm
- net SDA: track 7.60 -> 10.4 mm
- net SYSPOWER_IN: track 21.4 -> 20.9 mm
