File: Hardware/esp-oled-thing.sch (EAGLE design)
At the start: 44 parts, among them Q1 2.5A/30V, U1 MCP73831, U2 TPS61200

Commit message: parts ordered from Digikey,BOM added. Change quantity before ordering.
Parts:
- C1: value 10uF -> 10uF 10V
- C2, C7: value 0.1uF -> 0.1uF 10V
- C3, C4: value 4.7uF -> 4.7uF 10V
- C8: value 22uF -> 22uF 10V
- Q1: value 2.5A/30V -> DMP1045U
Changed lines of the file:
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@@
 <part name="P+1" library="SparkFun" deviceset="VCC" device=""/>
 <part name="D3" library="SparkFun-DiscreteSemi" deviceset="DIODE-SCHOTTKY" device="-BAT20J" value="BAT20J"/>
-<part name="Q1" library="SparkFun-DiscreteSemi" deviceset="MOSFET-PCHANNEL" device="DMG2307L" value="2.5A/30V"/>
+<part name="Q1" library="SparkFun-DiscreteSemi" deviceset="MOSFET-PCHANNEL" device="DMG2307L" value="DMP1045U"/>
 <part name="R12" library="adafruit" deviceset="R-US_" device="M0805" value="10K"/>
 <part name="GND3" library="supply1" deviceset="GND" device=""/>
@@
 </part>
 <part name="GND16" library="supply1" deviceset="GND" device=""/>
-<part name="C1" library="rcl" deviceset="C-US" device="C0805" value="10uF"/>
-<part name="C2" library="rcl" deviceset="C-US" device="C0805" value="0.1uF"/>
-<part name="C7" library="rcl" deviceset="C-US" device="C0805" value="0.1uF"/>
-<part name="C8" library="rcl" deviceset="C-US" device="C0805" value="22uF"/>
+<part name="C1" library="rcl" deviceset="C-US" device="C0805" value="10uF 10V"/>
+<part name="C2" library="rcl" deviceset="C-US" device="C0805" value="0.1uF 10V"/>
+<part name="C7" library="rcl" deviceset="C-US" device="C0805" value="0.1uF 10V"/>
+<part name="C8" library="rcl" deviceset="C-US" device="C0805" value="22uF 10V"/>
 <part name="R5" library="adafruit" deviceset="R-US_" device="M0805" value="10K"/>
 <part name="R17" library="adafruit" deviceset="R-US_" device="M0805" value="220K"/>
@@
 <part name="R23" library="adafruit" deviceset="R-US_" device="M0805" value="470E"/>
 <part name="R7" library="adafruit" deviceset="R-US_" device="M0805" value="2K"/>
-<part name="C3" library="rcl" deviceset="C-US" device="C0805" value="4.7uF"/>
-<part name="C4" library="rcl" deviceset="C-US" device="C0805" value="4.7uF"/>
+<part name="C3" library="rcl" deviceset="C-US" device="C0805" value="4.7uF 10V"/>
+<part name="C4" library="rcl" deviceset="C-US" device="C0805" value="4.7uF 10V"/>
 </parts>
 <sheets>
